File: Matchstick 2.0.brd (EAGLE design)
At the start: 73 x 38 mm, 13 parts, among them IC1 74HCT125D, J1 694106301002, J2 TARGET, J3 691241510006, J4 691241510006, U1 M5STAMP PICO

Commit message: updated silk screen
Parts:
- renumbered D17 to D1
Other:
- board text added: "S1 - G0 S2 - G33 D1 - G22"
Changed lines of the file:
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@@
 <grid distance="1" unitdist="mm" unit="mm" style="lines" multiple="1" display="yes" altdistance="5" altunitdist="mil" altunit="mil"/>
 <layers>
-<layer number="1" name="Top" color="4" fill="1" visible="yes" active="yes"/>
+<layer number="1" name="Top" color="4" fill="1" visible="no" active="yes"/>
 <layer number="16" name="Bottom" color="1" fill="1" visible="yes" active="yes"/>
 <layer number="17" name="Pads" color="2" fill="1" visible="yes" active="yes"/>
@@
 <layer number="19" name="Unrouted" color="6" fill="1" visible="yes" active="yes"/>
 <layer number="20" name="Dimension" color="24" fill="1" visible="yes" active="yes"/>
-<layer number="21" name="tPlace" color="7" fill="1" visible="yes" active="yes"/>
+<layer number="21" name="tPlace" color="7" fill="1" visible="no" active="yes"/>
 <layer number="22" name="bPlace" color="7" fill="1" visible="yes" active="yes"/>
-<layer number="23" name="tOrigins" color="15" fill="1" visible="yes" active="yes"/>
+<layer number="23" name="tOrigins" color="15" fill="1" visible="no" active="yes"/>
 <layer number="24" name="bOrigins" color="15" fill="1" visible="yes" active="yes"/>
-<layer number="25" name="tNames" color="7" fill="1" visible="yes" active="yes"/>
+<layer number="25" name="tNames" color="7" fill="1" visible="no" active="yes"/>
 <layer number="26" name="bNames" color="7" fill="1" visible="yes" active="yes"/>
 <layer number="27" name="tValues" color="7" fill="1" visible="no" active="yes"/>
@@
 <layer number="37" name="tTest" color="7" fill="1" visible="no" active="yes"/>
 <layer number="38" name="bTest" color="7" fill="1" visible="no" active="yes"/>
-<layer number="39" name="tKeepout" color="4" fill="11" visible="yes" active="yes"/>
+<layer number="39" name="tKeepout" color="4" fill="11" visible="no" active="yes"/>
 <layer number="40" name="bKeepout" color="1" fill="11" visible="yes" active="yes"/>
-<layer number="41" name="tRestrict" color="4" fill="10" visible="yes" active="yes"/>
+<layer number="41" name="tRestrict" color="4" fill="10" visible="no" active="yes"/>
 <layer number="42" name="bRestrict" color="1" fill="10" visible="yes" active="yes"/>
 <layer number="43" name="vRestrict" color="2" fill="10" visible="no" active="yes"/>
@@
 <layer number="49" name="Reference" color="7" fill="1" visible="no" active="yes"/>
 <layer number="50" name="dxf" color="7" fill="1" visible="no" active="no"/>
-<layer number="51" name="tDocu" color="7" fill="1" visible="yes" active="yes"/>
+<layer number="51" name="tDocu" color="7" fill="1" visible="no" active="yes"/>
 <layer number="52" name="bDocu" color="7" fill="1" visible="yes" active="yes"/>
 <layer number="53" name="tGND_GNDA" color="7" fill="9" visible="no" active="no"/>
@@
 <text x="26" y="27" size="2.54" layer="21" ratio="12" align="top-center">CH3</text>
 <text x="11" y="27" size="2.54" layer="21" ratio="12" align="top-center">CH4</text>
+<text x="55.016" y="25.238" size="1.27" layer="22" rot="MR0">S1 - G0
+S2 - G33
+D1 - G22</text>
 </plain>
 <attributes>
@@
 <attribute name="VOLTAGE_RATING" value="" x="-37.77" y="43.13" size="1.778" layer="28" rot="MR90" display="off"/>
 </element>
-<element name="D17" library="LED" library_urn="urn:adsk.eagle:library:22900745" package="LEDC2012X110N_FLAT-R" package3d_urn="urn:adsk.eagle:package:24294806/1" value="LED_RED" x="50" y="19" smashed="yes" rot="MR270">
+<element name="D1" library="LED" library_urn="urn:adsk.eagle:library:22900745" package="LEDC2012X110N_FLAT-R" package3d_urn="urn:adsk.eagle:package:24294806/1" value="LED_RED" x="50" y="19" smashed="yes" rot="MR270">
 <attribute name="CATEGORY" value="LED" x="113.5" y="-22.91" size="1.778" layer="28" rot="MR270" display="off"/>
 <attribute name="COLOR" value="RED" x="113.5" y="-22.91" size="1.778" layer="28" rot="MR270" display="off"/>
@@
 <signal name="SATUS_LED$1">
 <contactref element="U1" pad="6"/>
-<contactref element="D17" pad="A"/>
+<contactref element="D1" pad="A"/>
 <via x="40.27" y="16.46" extent="1-16" drill="0.35"/>
 <wire x1="36.5" y1="16.46" x2="40.27" y2="16.46" width="0.508" layer="1"/>
@@
 </signal>
 <signal name="SATUS_LED$2">
-<contactref element="D17" pad="C"/>
+<contactref element="D1" pad="C"/>
 <contactref element="R1" pad="1"/>
 <wire x1="45" y1="19.9195" x2="45.1055" y2="20.025" width="0.508" layer="16"/>
