File: Matchstick 2.0.sch (EAGLE design)
At the start: 13 parts, among them IC1 74HCT125D, J1 694106301002, J2 TARGET, J3 691241510006, J4 691241510006, U1 M5STAMP PICO

Commit message: updated silk screen
Parts:
- renumbered D17 to D1
Changed lines of the file:
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@@
 <drawing>
 <settings>
-<setting alwaysvectorfont="no"/>
+<setting alwaysvectorfont="yes"/>
 <setting verticaltext="up"/>
 </settings>
-<grid distance="1" unitdist="mm" unit="mm" style="lines" multiple="1" display="yes" altdistance="1" altunitdist="mm" altunit="mm"/>
+<grid distance="0.1" unitdist="inch" unit="inch" style="lines" multiple="1" display="no" altdistance="0.01" altunitdist="inch" altunit="inch"/>
 <layers>
 <layer number="1" name="Top" color="4" fill="1" visible="no" active="no"/>
@@
 <part name="FRAME1" library="frames" library_urn="urn:adsk.eagle:library:229" deviceset="DINA5_L" device="" value="ESP32 PICO"/>
 <part name="S1" library="SparkFun-Switches" library_urn="urn:adsk.eagle:library:535" deviceset="MOMENTARY-SWITCH-SPST" device="-SMD-5.2MM" package3d_urn="urn:adsk.eagle:package:40167/1" value="FLASH"/>
-<part name="D17" library="LED" library_urn="urn:adsk.eagle:library:22900745" deviceset="CHIP-FLAT-R" device="_0805" package3d_urn="urn:adsk.eagle:package:24294806/1" value="LED_RED"/>
+<part name="D1" library="LED" library_urn="urn:adsk.eagle:library:22900745" deviceset="CHIP-FLAT-R" device="_0805" package3d_urn="urn:adsk.eagle:package:24294806/1" value="LED_RED"/>
 <part name="R1" library="Resistor" library_urn="urn:adsk.eagle:library:16378527" deviceset="R-US" device="CHIP-0805(2012-METRIC)" package3d_urn="urn:adsk.eagle:package:16378559/2" technology="_" value="330"/>
 <part name="J2" library="custom" library_urn="urn:adsk.eagle:library:28163416" deviceset="6_PIN_SERIAL_TARGET" device="SILK" package3d_urn="urn:adsk.eagle:package:37733454/1" value="TARGET"/>
@@
 <attribute name="VALUE" x="134.84" y="56.15" size="1.778" layer="96" font="vector" align="top-center"/>
 </instance>
-<instance part="D17" gate="G$1" x="119.6" y="75.2" smashed="yes" rot="R90">
+<instance part="D1" gate="G$1" x="119.6" y="75.2" smashed="yes" rot="R90">
 <attribute name="NAME" x="119.854" y="72.152" size="1.778" layer="95" align="top-right"/>
 <attribute name="VALUE" x="115.79" y="67.58" size="1.778" layer="96" rot="R180" align="top-right"/>
@@
 <segment>
 <pinref part="U1" gate="G$1" pin="G22"/>
-<pinref part="D17" gate="G$1" pin="A"/>
+<pinref part="D1" gate="G$1" pin="A"/>
 <wire x1="101.82" y1="75.2" x2="117.06" y2="75.2" width="0.1524" layer="91"/>
 </segment>
@@
 <net name="SATUS_LED$2" class="0">
 <segment>
-<pinref part="D17" gate="G$1" pin="C"/>
+<pinref part="D1" gate="G$1" pin="C"/>
 <pinref part="R1" gate="G$1" pin="1"/>
 <wire x1="124.68" y1="75.2" x2="129.76" y2="75.2" width="0.1524" layer="91"/>

Commit message: changed signal traces to 0.254mm
Connections:
- net GND renamed STATUS_LED$2
Changed lines of the file:
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@@
 <drawing>
 <settings>
-<setting alwaysvectorfont="yes"/>
+<setting alwaysvectorfont="no"/>
 <setting verticaltext="up"/>
 </settings>
@@
 </busses>
 <nets>
-<net name="GND" class="0">
+<net name="STATUS_LED$2" class="0">
 <segment>
 <pinref part="U1" gate="G$1" pin="GND@1"/>

Commit message: fixing the crossed signals
Connections:
- new net GND: C2.-, IC1A.OE, IC1B.OE, IC1C.OE, IC1D.OE, J1.2, J2.GND, J3.3, J3.6, J4.3, J4.6, R1.2, R2.1, S1.1, U1.GND@1, U1.GND@2, U1.GND@3
- net STATUS_LED$2: no longer C2.-, IC1A.OE, IC1B.OE, IC1C.OE, IC1D.OE, J1.2, J2.GND, J3.3, J3.6, J4.3, J4.6, R1.2, R2.1, S1.1, U1.GND@1, U1.GND@2, U1.GND@3
Changed lines of the file:
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@@
 <drawing>
 <settings>
-<setting alwaysvectorfont="no"/>
+<setting alwaysvectorfont="yes"/>
 <setting verticaltext="up"/>
 </settings>
@@
 <net name="STATUS_LED$2" class="0">
 <segment>
-<pinref part="U1" gate="G$1" pin="GND@1"/>
-<wire x1="101.82" y1="67.58" x2="104.36" y2="67.58" width="0.1524" layer="91"/>
-<label x="104.36" y="67.58" size="0.8128" layer="95" xref="yes"/>
-</segment>
-<segment>
-<wire x1="117.06" y1="32.02" x2="117.06" y2="35.83" width="0.1524" layer="91"/>
-<label x="117.06" y="35.83" size="0.8128" layer="95" rot="MR0" xref="yes"/>
-<pinref part="J2" gate="G$1" pin="GND"/>
-</segment>
-<segment>
-<pinref part="S1" gate="G$1" pin="1"/>
-<wire x1="139.92" y1="52.34" x2="146.24" y2="52.34" width="0.1524" layer="91"/>
-<label x="146.24" y="52.34" size="0.8128" layer="95" xref="yes"/>
-</segment>
-<segment>
-<pinref part="U1" gate="G$1" pin="GND@2"/>
-<wire x1="101.82" y1="65.04" x2="104.36" y2="65.04" width="0.1524" layer="91"/>
-<label x="104.36" y="65.04" size="0.8128" layer="95" xref="yes"/>
-</segment>
-<segment>
-<pinref part="U1" gate="G$1" pin="GND@3"/>
-<wire x1="101.82" y1="54.88" x2="104.36" y2="54.88" width="0.1524" layer="91"/>
-<label x="104.36" y="54.88" size="0.8128" layer="95" xref="yes"/>
-</segment>
-<segment>
-<pinref part="R1" gate="G$1" pin="2"/>
-<wire x1="139.92" y1="75.2" x2="146.24" y2="75.2" width="0.1524" layer="91"/>
-<label x="146.24" y="75.2" size="0.8128" layer="95" xref="yes"/>
-</segment>
-<segment>
-<wire x1="24.32" y1="77.64" x2="21.78" y2="77.64" width="0.1524" layer="91"/>
-<label x="21.78" y="77.64" size="0.8128" layer="95" rot="R180" xref="yes"/>
-<pinref part="IC1" gate="A" pin="OE"/>
-</segment>
-<segment>
-<wire x1="24.32" y1="59.86" x2="21.78" y2="59.86" width="0.1524" layer="91"/>
-<label x="21.78" y="59.86" size="0.8128" layer="95" rot="R180" xref="yes"/>
-<pinref part="IC1" gate="B" pin="OE"/>
-</segment>
-<segment>
 <pinref part="IC1" gate="P" pin="GND"/>
 <pinref part="SUPPLY2" gate="G$1" pin="GND"/>
@@
 <junction x="-8.7" y="54.78"/>
 </segment>
-<segment>
-<pinref part="IC1" gate="C" pin="OE"/>
-<wire x1="63.66" y1="77.64" x2="61.12" y2="77.64" width="0.1524" layer="91"/>
-<label x="61.12" y="77.64" size="0.8128" layer="95" rot="R180" xref="yes"/>
-</segment>
-<segment>
-<pinref part="IC1" gate="D" pin="OE"/>
-<wire x1="63.66" y1="59.86" x2="61.12" y2="59.86" width="0.1524" layer="91"/>
-<label x="61.12" y="59.86" size="0.8128" layer="95" rot="R180" xref="yes"/>
-</segment>
-<segment>
-<pinref part="J1" gate="G$1" pin="2"/>
-<wire x1="126.34" y1="93.58" x2="129.8" y2="93.58" width="0.1524" layer="91"/>
-<label x="129.8" y="93.66" size="0.8128" layer="95" xref="yes"/>
-</segment>
-<segment>
-<pinref part="R2" gate="G$1" pin="1"/>
-<wire x1="101.6" y1="17.78" x2="104.14" y2="17.78" width="0.1524" layer="91"/>
-<label x="104.14" y="17.78" size="0.8128" layer="95" xref="yes"/>
-</segment>
-<segment>
-<wire x1="12.7" y1="20.32" x2="15.24" y2="20.32" width="0.1524" layer="91"/>
-<label x="15.24" y="20.32" size="0.8128" layer="95" rot="MR180" xref="yes"/>
-<pinref part="J3" gate="G$1" pin="3"/>
-</segment>
-<segment>
-<wire x1="33.02" y1="17.78" x2="30.48" y2="17.78" width="0.1524" layer="91"/>
-<label x="30.48" y="17.78" size="0.8128" layer="95" rot="MR0" xref="yes"/>
-<pinref part="J4" gate="G$1" pin="3"/>
-</segment>
-<segment>
-<pinref part="C2" gate="G$1" pin="-"/>
-<wire x1="137.7" y1="92.44" x2="137.7" y2="89.9" width="0.1524" layer="91"/>
-<label x="137.7" y="89.9" size="0.8128" layer="95" rot="R270" xref="yes"/>
-</segment>
-<segment>
-<wire x1="12.7" y1="12.7" x2="15.24" y2="12.7" width="0.1524" layer="91"/>
-<label x="15.24" y="12.7" size="0.8128" layer="95" rot="MR180" xref="yes"/>
-<pinref part="J3" gate="G$1" pin="6"/>
-</segment>
-<segment>
-<wire x1="33.02" y1="25.4" x2="30.48" y2="25.4" width="0.1524" layer="91"/>
-<label x="30.48" y="25.4" size="0.8128" layer="95" rot="MR0" xref="yes"/>
-<pinref part="J4" gate="G$1" pin="6"/>
-</segment>
 </net>
 <net name="DATA$4" class="0">
@@
 </segment>
 </net>
+<net name="GND" class="0">
+<segment>
+<wire x1="24.32" y1="77.64" x2="21.78" y2="77.64" width="0.1524" layer="91"/>
+<label x="21.78" y="77.64" size="0.8128" layer="95" rot="R180" xref="yes"/>
+<pinref part="IC1" gate="A" pin="OE"/>
+</segment>
+<segment>
+<pinref part="IC1" gate="C" pin="OE"/>
+<wire x1="63.66" y1="77.64" x2="61.12" y2="77.64" width="0.1524" layer="91"/>
+<label x="61.12" y="77.64" size="0.8128" layer="95" rot="R180" xref="yes"/>
+</segment>
+<segment>
+<pinref part="IC1" gate="D" pin="OE"/>
+<wire x1="63.66" y1="59.86" x2="61.12" y2="59.86" width="0.1524" layer="91"/>
+<label x="61.12" y="59.86" size="0.8128" layer="95" rot="R180" xref="yes"/>
+</segment>
+<segment>
+<wire x1="24.32" y1="59.86" x2="21.78" y2="59.86" width="0.1524" layer="91"/>
+<label x="21.78" y="59.86" size="0.8128" layer="95" rot="R180" xref="yes"/>
+<pinref part="IC1" gate="B" pin="OE"/>
+</segment>
+<segment>
+<pinref part="J1" gate="G$1" pin="2"/>
+<wire x1="126.34" y1="93.58" x2="129.8" y2="93.58" width="0.1524" layer="91"/>
+<label x="129.8" y="93.66" size="0.8128" layer="95" xref="yes"/>
+</segment>
+<segment>
+<pinref part="C2" gate="G$1" pin="-"/>
+<wire x1="137.7" y1="92.44" x2="137.7" y2="89.9" width="0.1524" layer="91"/>
+<label x="137.7" y="89.9" size="0.8128" layer="95" rot="R270" xref="yes"/>
+</segment>
+<segment>
+<pinref part="R1" gate="G$1" pin="2"/>
+<wire x1="139.92" y1="75.2" x2="146.24" y2="75.2" width="0.1524" layer="91"/>
+<label x="146.24" y="75.2" size="0.8128" layer="95" xref="yes"/>
+</segment>
+<segment>
+<pinref part="S1" gate="G$1" pin="1"/>
+<wire x1="139.92" y1="52.34" x2="146.24" y2="52.34" width="0.1524" layer="91"/>
+<label x="146.24" y="52.34" size="0.8128" layer="95" xref="yes"/>
+</segment>
+<segment>
+<wire x1="117.06" y1="32.02" x2="117.06" y2="35.83" width="0.1524" layer="91"/>
+<label x="117.06" y="35.83" size="0.8128" layer="95" rot="MR0" xref="yes"/>
+<pinref part="J2" gate="G$1" pin="GND"/>
+</segment>
+<segment>
+<pinref part="R2" gate="G$1" pin="1"/>
+<wire x1="101.6" y1="17.78" x2="104.14" y2="17.78" width="0.1524" layer="91"/>
+<label x="104.14" y="17.78" size="0.8128" layer="95" xref="yes"/>
+</segment>
+<segment>
+<wire x1="33.02" y1="25.4" x2="30.48" y2="25.4" width="0.1524" layer="91"/>
+<label x="30.48" y="25.4" size="0.8128" layer="95" rot="MR0" xref="yes"/>
+<pinref part="J4" gate="G$1" pin="6"/>
+</segment>
+<segment>
+<wire x1="33.02" y1="17.78" x2="30.48" y2="17.78" width="0.1524" layer="91"/>
+<label x="30.48" y="17.78" size="0.8128" layer="95" rot="MR0" xref="yes"/>
+<pinref part="J4" gate="G$1" pin="3"/>
+</segment>
+<segment>
+<wire x1="12.7" y1="12.7" x2="15.24" y2="12.7" width="0.1524" layer="91"/>
+<label x="15.24" y="12.7" size="0.8128" layer="95" rot="MR180" xref="yes"/>
+<pinref part="J3" gate="G$1" pin="6"/>
+</segment>
+<segment>
+<wire x1="12.7" y1="20.32" x2="15.24" y2="20.32" width="0.1524" layer="91"/>
+<label x="15.24" y="20.32" size="0.8128" layer="95" rot="MR180" xref="yes"/>
+<pinref part="J3" gate="G$1" pin="3"/>
+</segment>
+<segment>
+<pinref part="U1" gate="G$1" pin="GND@1"/>
+<wire x1="101.82" y1="67.58" x2="104.36" y2="67.58" width="0.1524" layer="91"/>
+<label x="104.36" y="67.58" size="0.8128" layer="95" xref="yes"/>
+</segment>
+<segment>
+<pinref part="U1" gate="G$1" pin="GND@2"/>
+<wire x1="101.82" y1="65.04" x2="104.36" y2="65.04" width="0.1524" layer="91"/>
+<label x="104.36" y="65.04" size="0.8128" layer="95" xref="yes"/>
+</segment>
+<segment>
+<pinref part="U1" gate="G$1" pin="GND@3"/>
+<wire x1="101.82" y1="54.88" x2="104.36" y2="54.88" width="0.1524" layer="91"/>
+<label x="104.36" y="54.88" size="0.8128" layer="95" xref="yes"/>
+</segment>
+</net>

Commit message: fixing the crossed signals 2
Connections:
- removed net STATUS_LED$2: C1.2, IC1P.GND
- net GND: now also C1.2, IC1P.GND

Commit message: updated readme with schematic
Parts:
- C2: value (none) -> 1000 uF
Changed lines of the file:
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@@
 <part name="J3" library="Wurth_Connectors_WR-TBL Rising Cage Clamp" library_urn="urn:adsk.eagle:library:16280519" deviceset="691241510006" device="" package3d_urn="urn:adsk.eagle:package:16248563/2"/>
 <part name="J4" library="Wurth_Connectors_WR-TBL Rising Cage Clamp" library_urn="urn:adsk.eagle:library:16280519" deviceset="691241510006" device="" package3d_urn="urn:adsk.eagle:package:16248563/2"/>
-<part name="C2" library="Capacitor" library_urn="urn:adsk.eagle:library:16290819" deviceset="C-POL" device="RADIAL-11MM-DIA" package3d_urn="urn:adsk.eagle:package:16290899/1" technology="_"/>
+<part name="C2" library="Capacitor" library_urn="urn:adsk.eagle:library:16290819" deviceset="C-POL" device="RADIAL-11MM-DIA" package3d_urn="urn:adsk.eagle:package:16290899/1" technology="_" value="1000 uF"/>
 </parts>
 <sheets>
